Commit message: Corrected moveit_config folder

File: poke_description/urdf/poke.urdf.xacro (robot description, xacro)
@@ -5,5 +5,5 @@
                                    Export urdf to pdf:  $ urdf_to_graphiz poke.urdf
 -->
-<robot name="poke_arm" xmlns:xacro="http://ros.org/wiki/xacro"
+<robot name="poke_arm_main" xmlns:xacro="http://ros.org/wiki/xacro"
     xmlns:sensor="http://playerstage.sourceforge.net/gazebo/xmlschema/#sensor"
     xmlns:controller="http://playerstage.sourceforge.net/gazebo/xmlschema/#controller"
@@ -11,13 +11,15 @@
     <!-- Included URDF Files -->
     <xacro:include filename="$(find poke_description)/urdf/poke.xacro" />
+    <!--
+    For simulating only the arm, we'll use "world" as the link name.
+    For using it on the turtlebot, use "base_link" as the link name.
+    -->
     <!-- As we don't have here a turtlebot, add a base_link link as its location reference -->
-    <link name="base_link"/>
-    <!-- Poke arm macro: we can configure joints velocity limit and lower/upper limits
-         for the first joint (arm_shoulder_pan) to allow accessing to different operational
-         areas, e.g. left handed vs. right handed robot -->
-    <poke_arm parent="base_link" color="white" joints_vlimit="1.571">
-      <!-- Place the "floating" arm at the location it should be if mounted on a turtlebot,
-           as pick and place and other demos assume this location -->
-      <origin xyz="0.1 0.03 0.435"/>
+    <link name="world"/>
+    <!-- Poke arm macro: we can configure joints velocity limit -->
+    <poke_arm parent="world" color="white" joints_vlimit="1.571">
+      <!-- Place the "floating" arm at the location it should be if mounted on a turtlebot -->
+      <!-- origin xyz="0.1 0.03 0.435"/-->
+      <origin xyz="0 0 0"/>
     </poke_arm>
 </robot>

File: poke_description/urdf/poke.xacro (robot description, xacro)
@@ -61,4 +61,5 @@
   <mtrT jointName="p1_joint"/>
   <mtrT jointName="p2_joint"/>
+  <mtrT jointName="p3_joint"/>
   </xacro:macro>
 </robot>

File: poke_description/urdf/poke_hardware.xacro (robot description, xacro)
@@ -130,4 +130,5 @@
   <xacro:macro name="cSeg" params="parent name color">
     <joint name="${name}_joint" type="continuous">
+      <axis xyz="0 0 1" />
       <parent link="${parent}"/>
       <child link="${name}_link" />
